File: pcb/I2C.sch (KiCad schematic (older format))
At the start: 12 parts, among them U10 PCF8523TK, Y1 ABS06-107-32.768KHZ-T

Commit message: Added components dikey part numbers in modified sheets
Parts:
- C23, C25: DigiKey (none) -> 1276-1599-1-ND
- C24: DigiKey (none) -> 493-4330-ND
- C26: DigiKey (none) -> 1276-1442-1-ND
- D7: DigiKey (none) -> 1SS389L3FCT-ND
- R10: DigiKey (none) -> P453LCT-ND
- R12: DigiKey (none) -> P499LCT-ND
- R13: DigiKey (none) -> P100LCT-ND
- R14, R15: DigiKey (none) -> P2.20KLCT-ND
- U10: DigiKey (none) -> 568-6648-1-ND
- Y1: DigiKey (none) -> 535-12373-1-ND
Changed lines of the file:
@@
 F 2 "SMD:HVSON8" H 5775 2525 50  0001 C CNN
 F 3 "" H 5775 2525 50  0001 C CNN
+F 4 "568-6648-1-ND" H 6075 2425 50  0001 C CNN "DigiKey"
 	1    6075 2425
 	1    0    0    -1
@@
 F 2 "Capacitor_THT:CP_Radial_D6.3mm_P2.50mm" H 5350 2650 50  0001 C CNN
 F 3 "~" H 5350 2650 50  0001 C CNN
+F 4 "493-4330-ND" H 5350 2650 50  0001 C CNN "DigiKey"
 	1    5350 2650
 	1    0    0    -1
@@
 F 2 "Resistor_SMD:R_0402_1005Metric" H 5125 2475 50  0001 C CNN
 F 3 "~" H 5125 2475 50  0001 C CNN
+F 4 "P100LCT-ND" V 5125 2475 50  0001 C CNN "DigiKey"
 	1    5125 2475
 	0    1    1    0
@@
 F 2 "Diode_SMD:D_SOD-523" V 4825 2475 50  0001 C CNN
 F 3 "~" V 4825 2475 50  0001 C CNN
+F 4 "1SS389L3FCT-ND" H 4825 2475 50  0001 C CNN "DigiKey"
 	1    4825 2475
 	-1   0    0    1
@@
 F 2 "Resistor_SMD:R_0402_1005Metric" H 4550 2275 50  0001 C CNN
 F 3 "~" H 4550 2275 50  0001 C CNN
+F 4 "P453LCT-ND" H 4550 2275 50  0001 C CNN "DigiKey"
 	1    4550 2275
 	-1   0    0    1
@@
 F 2 "Resistor_SMD:R_0402_1005Metric" H 4550 2650 50  0001 C CNN
 F 3 "~" H 4550 2650 50  0001 C CNN
+F 4 "P499LCT-ND" H 4550 2650 50  0001 C CNN "DigiKey"
 	1    4550 2650
 	-1   0    0    1
@@
 F 2 "SMD:ABS06-107" H 5500 1875 50  0001 C CNN
 F 3 "~" H 5500 1875 50  0001 C CNN
+F 4 "535-12373-1-ND" H 5500 1875 50  0001 C CNN "DigiKey"
 	1    5500 1875
 	1    0    0    -1
@@
 F 2 "Resistor_SMD:R_0402_1005Metric" H 6725 2775 50  0001 C CNN
 F 3 "~" H 6725 2775 50  0001 C CNN
+F 4 "P2.20KLCT-ND" H 6725 2775 50  0001 C CNN "DigiKey"
 	1    6725 2775
 	1    0    0    -1
@@
 F 2 "Resistor_SMD:R_0402_1005Metric" H 7050 2775 50  0001 C CNN
 F 3 "~" H 7050 2775 50  0001 C CNN
+F 4 "P2.20KLCT-ND" H 7050 2775 50  0001 C CNN "DigiKey"
 	1    7050 2775
 	1    0    0    -1
@@
 F 2 "Capacitor_SMD:C_0402_1005Metric" H 6825 2275 50  0001 C CNN
 F 3 "~" H 6825 2275 50  0001 C CNN
+F 4 "1276-1442-1-ND" H 6825 2275 50  0001 C CNN "DigiKey"
 	1    6825 2275
 	0    1    1    0
@@
 F 2 "Capacitor_SMD:C_0402_1005Metric" H 5250 1875 50  0001 C CNN
 F 3 "~" H 5250 1875 50  0001 C CNN
+F 4 "1276-1599-1-ND" H 5250 1875 50  0001 C CNN "DigiKey"
 	1    5250 1875
 	0    -1   -1   0
@@
 F 2 "Capacitor_SMD:C_0402_1005Metric" H 5750 1875 50  0001 C CNN
 F 3 "~" H 5750 1875 50  0001 C CNN
+F 4 "1276-1599-1-ND" H 5750 1875 50  0001 C CNN "DigiKey"
 	1    5750 1875
 	0    -1   -1   0
