File: pcb/stm32.sch (KiCad schematic (older format))
At the start: 40 parts, among them U11 LT1117CST-3.3, U401 STM32F100RBT6B, U485 SP481, X401 12MHz, Y2 Crystal

Commit message: Adición del STM32F4
Parts:
- C401, C402, C403, C404, C405, C406, C407, C410, C411, C74, C75, C76, CCS1, CHB1, CMB1, CRS1, CRs2, CS2, VCA1: symbol C -> chip_media-rescue:C
- CS1: symbol TCS3404 -> chip_media-rescue:TCS3404
- D8, D9: symbol LED -> chip_media-rescue:LED
- EXT1: symbol CONN_8X2M90 -> chip_media-rescue:CONN_8X2M90
- L1, L2: symbol L -> chip_media-rescue:L
- MB1: symbol CONN_3X1F -> chip_media-rescue:CONN_3X1F
- PEC1, PPH1: symbol BNC -> chip_media-rescue:BNC
- R33, R5, RMB1, RST2, RST3, RST4, RST5: symbol R -> chip_media-rescue:R
- U11: symbol LT1117CST -> chip_media-rescue:LT1117CST
- U401: symbol STM32F100RBTx -> chip_media-rescue:STM32F100RBTx
- U485: symbol SP481 -> chip_media-rescue:SP481
- X401: symbol ABM8G -> chip_media-rescue:ABM8G
- Y2: symbol Crystal -> chip_media-rescue:Crystal
Connections:
- wire segments 192 -> 223
