File: pcb/SensorShield.sch (KiCad schematic (older format))
At the start: 58 parts, among them U14 ICE40UP5K-SG48ITR, U15 GD25Q32CTIGR-Memory_Flash

Commit message: routing....
Parts:
- C50: footprint Resistor_SMD:R_0402_1005Metric -> Resistor_SMD:R_0603_1608Metric
- R29, R32, R33, R34, R5: footprint Resistor_SMD:R_0603_1608Metric -> Resistor_SMD:R_0402_1005Metric
Connections:
- net 1V2_ICE: now also U14.5 (VCC)
- net I2C_CLK_4: now also U14.4 (IOB_8a); no longer U14.40 (RGB1)
- net I2C_SDA_4: now also U14.3 (IOB_9b); no longer U14.39 (RGB0)
- net SPI_CLK: now also U14.39 (RGB0)
- net SPI_CS_4: now also U14.48 (IOB_4a); no longer U14.41 (RGB2)
- net SPI_MISO: now also U14.2 (IOB_6a)
- net SPI_MOSI: now also U14.40 (RGB1)
- net VCC_PLL: now also U14.29 (VCCPLL); no longer U14.5 (VCC)
Changed lines of the file:
@@
 AR Path="/5E9C016D/5E9D8A4E" Ref="U14"  Part="4"
 F 0 "U14" V 2267 5600 50  0000 C CNN
-F 1 "ICE40UP5K-SG48ITR" V 2176 5600 50  0000 C CNN
+F 1 "ICE40UP5K-SG48ITR" V 1650 5600 50  0000 C CNN
 F 2 "Package_DFN_QFN:QFN-48-1EP_7x7mm_P0.5mm_EP5.6x5.6mm" H 1900 4250 50  0001 C CNN
 F 3 "" H 1500 6600 50  0001 C CNN
@@
 Wire Wire Line
 	6200 1950 6700 1950
-Text Label 1050 5500 0    50   ~ 0
+Text Label 1050 5400 0    50   ~ 0
 VCC_PLL
 Wire Wire Line
-	1050 5500 1500 5500
+	1050 5400 1500 5400
 Wire Wire Line
 	2400 2450 2850 2450
@@
 F 0 "R32" V 3293 5400 50  0000 C CNN
 F 1 "100" V 3384 5400 50  0000 C CNN
-F 2 "Resistor_SMD:R_0603_1608Metric" V 3430 5400 50  0001 C CNN
+F 2 "Resistor_SMD:R_0402_1005Metric" V 3430 5400 50  0001 C CNN
 F 3 "~" H 3500 5400 50  0001 C CNN
 	1    3500 5400
@@
 F 0 "C50" H 4415 5596 50  0000 L CNN
 F 1 "4.7u" H 4415 5505 50  0000 L CNN
-F 2 "Resistor_SMD:R_0402_1005Metric" H 4338 5400 50  0001 C CNN
+F 2 "Resistor_SMD:R_0603_1608Metric" H 4338 5400 50  0001 C CNN
 F 3 "~" H 4300 5550 50  0001 C CNN
 	1    4300 5550
@@
 AR Path="/5E98CC69/5E9ECB99/5E9D8B37" Ref="R33"  Part="1"
 AR Path="/5E9C016D/5E9D8B37" Ref="R33"  Part="1"
+AR Path="/5E96F696/5E9D8B37" Ref="R33"  Part="1"
 F 0 "R33" H 4430 8004 50  0000 R CNN
 F 1 "10K" H 4430 8095 50  0000 R CNN
-F 2 "Resistor_SMD:R_0603_1608Metric" V 4430 8050 50  0001 C CNN
+F 2 "Resistor_SMD:R_0402_1005Metric" V 4430 8050 50  0001 C CNN
 F 3 "~" H 4500 8050 50  0001 C CNN
 	1    4500 8050
@@
 F 0 "R34" H 4730 8004 50  0000 R CNN
 F 1 "10K" H 4730 8095 50  0000 R CNN
-F 2 "Resistor_SMD:R_0603_1608Metric" V 4730 8050 50  0001 C CNN
+F 2 "Resistor_SMD:R_0402_1005Metric" V 4730 8050 50  0001 C CNN
 F 3 "~" H 4800 8050 50  0001 C CNN
 	1    4800 8050
@@
 F 0 "R29" H 2380 8054 50  0000 R CNN
 F 1 "10K" H 2380 8145 50  0000 R CNN
-F 2 "Resistor_SMD:R_0603_1608Metric" V 2380 8100 50  0001 C CNN
+F 2 "Resistor_SMD:R_0402_1005Metric" V 2380 8100 50  0001 C CNN
 F 3 "~" H 2450 8100 50  0001 C CNN
 	1    2450 8100
@@
 	4050 2450 4250 2450
 Wire Wire Line
-	1050 5600 1500 5600
-Text Label 1050 5600 0    50   ~ 0
+	1050 5500 1450 5500
+Text Label 1050 5500 0    50   ~ 0
 +1.2V_CORE
 Text Label 1300 6300 0    50   ~ 0
@@
 I2C_CLK_3
 Wire Wire Line
-	750  4050 1300 4050
+	5250 3150 5800 3150
 Wire Wire Line
-	750  3950 1300 3950
-Text Label 750  3950 0    50   ~ 0
+	5250 3250 5800 3250
+Text Label 5250 3250 0    50   ~ 0
 I2C_SDA_4
-Text Label 750  4050 0    50   ~ 0
+Text Label 5250 3150 0    50   ~ 0
 I2C_CLK_4
 Wire Wire Line
@@
 SPI_CS_0
 Wire Wire Line
-	1300 4150 750  4150
-Text Label 750  4150 0    50   ~ 0
+	5800 2850 5250 2850
+Text Label 5250 2850 0    50   ~ 0
 SPI_CS_4
 Wire Wire Line
@@
 F 0 "R5" H 2380 8554 50  0000 R CNN
 F 1 "10K" H 2380 8645 50  0000 R CNN
-F 2 "Resistor_SMD:R_0603_1608Metric" V 2380 8600 50  0001 C CNN
+F 2 "Resistor_SMD:R_0402_1005Metric" V 2380 8600 50  0001 C CNN
 F 3 "~" H 2450 8600 50  0001 C CNN
 	1    2450 8600
@@
 Text Label 750  2850 0    50   ~ 0
 I2C_CLK_8
+Wire Wire Line
+	1300 4050 750  4050
+Text Label 750  4050 0    50   ~ 0
+SPI_MOSI
+Text Label 750  3950 0    50   ~ 0
+SPI_CLK
+Wire Wire Line
+	1300 3950 750  3950
+Wire Wire Line
+	1525 5600 1500 5600
+Wire Wire Line
+	1450 5600 1450 5500
+Connection ~ 1500 5600
+Wire Wire Line
+	1500 5600 1450 5600
+Connection ~ 1450 5500
+Wire Wire Line
+	1450 5500 1500 5500
+Text Label 5250 3050 0    50   ~ 0
+SPI_MISO
+Wire Wire Line
+	5800 3050 5250 3050
 Wire Bus Line
 	2250 9700 2250 10200
