File: pcb/PSU.sch (KiCad schematic (older format))
At the start: 19 parts, among them Q3 DMG2305UX, Q4 BCM857BS, U18 XCL206B123, U9 XCL214B333

Commit message: power connector
Parts:
- added PWR1: Conn_01x03, TH:10142708-06200LF, symbol Connector_Generic:Conn_02x03_Odd_Even
Connections:
- net GND: now also PWR1.5 (Pin_5), PWR1.6 (Pin_6)
- net Vin: now also PWR1.1 (Pin_1), PWR1.2 (Pin_2)
Changed lines of the file:
@@
 Text Label 2750 1700 0    39   ~ 0
 L1_Lx_3V3
+$Comp
+L Connector_Generic:Conn_02x03_Odd_Even G?
+U 1 1 5EAC048F
+P 1500 3675
+AR Path="/5E9C016D/5EAC048F" Ref="G?"  Part="1"
+AR Path="/5EA61A2E/5EAC048F" Ref="PWR1"  Part="1"
+F 0 "PWR1" H 1450 3975 50  0000 L CNN
+F 1 "Conn_01x03" H 1580 3626 50  0001 L CNN
+F 2 "TH:10142708-06200LF" H 1500 3675 50  0001 C CNN
+F 3 "~" H 1500 3675 50  0001 C CNN
+	1    1500 3675
+	1    0    0    -1
+$EndComp
+$Comp
+L power:GND #PWR?
+U 1 1 5EAC0495
+P 1800 3775
+AR Path="/5E98CC69/5E9ECB99/5EAC0495" Ref="#PWR?"  Part="1"
+AR Path="/5E98CC69/5EA15EEE/5EAC0495" Ref="#PWR?"  Part="1"
+AR Path="/5E98CC69/5EA18277/5EAC0495" Ref="#PWR?"  Part="1"
+AR Path="/5E98CC69/5EA1A185/5EAC0495" Ref="#PWR?"  Part="1"
+AR Path="/5E98CC69/5EA1A18E/5EAC0495" Ref="#PWR?"  Part="1"
+AR Path="/5E98CC69/5EA1A197/5EAC0495" Ref="#PWR?"  Part="1"
+AR Path="/5E98CC69/5EA1B439/5EAC0495" Ref="#PWR?"  Part="1"
+AR Path="/5E98CC69/5EA1B442/5EAC0495" Ref="#PWR?"  Part="1"
+AR Path="/5E98CC69/5EA1B44B/5EAC0495" Ref="#PWR?"  Part="1"
+AR Path="/5E9C016D/5EAC0495" Ref="#PWR?"  Part="1"
+AR Path="/5EA61A2E/5EAC0495" Ref="#PWR0226"  Part="1"
+F 0 "#PWR0226" H 1800 3525 50  0001 C CNN
+F 1 "GND" H 1805 3602 50  0000 C CNN
+F 2 "" H 1800 3775 50  0001 C CNN
+F 3 "" H 1800 3775 50  0001 C CNN
+	1    1800 3775
+	1    0    0    -1
+$EndComp
+Wire Wire Line
+	1800 3575 1950 3575
+Text Label 1950 3575 2    60   ~ 0
+Vin
+$Comp
+L power:GND #PWR?
+U 1 1 5EA95F9E
+P 1300 3775
+AR Path="/5E98CC69/5E9ECB99/5EA95F9E" Ref="#PWR?"  Part="1"
+AR Path="/5E98CC69/5EA15EEE/5EA95F9E" Ref="#PWR?"  Part="1"
+AR Path="/5E98CC69/5EA18277/5EA95F9E" Ref="#PWR?"  Part="1"
+AR Path="/5E98CC69/5EA1A185/5EA95F9E" Ref="#PWR?"  Part="1"
+AR Path="/5E98CC69/5EA1A18E/5EA95F9E" Ref="#PWR?"  Part="1"
+AR Path="/5E98CC69/5EA1A197/5EA95F9E" Ref="#PWR?"  Part="1"
+AR Path="/5E98CC69/5EA1B439/5EA95F9E" Ref="#PWR?"  Part="1"
+AR Path="/5E98CC69/5EA1B442/5EA95F9E" Ref="#PWR?"  Part="1"
+AR Path="/5E98CC69/5EA1B44B/5EA95F9E" Ref="#PWR?"  Part="1"
+AR Path="/5E9C016D/5EA95F9E" Ref="#PWR?"  Part="1"
+AR Path="/5EA61A2E/5EA95F9E" Ref="#PWR?"  Part="1"
+F 0 "#PWR?" H 1300 3525 50  0001 C CNN
+F 1 "GND" H 1305 3602 50  0000 C CNN
+F 2 "" H 1300 3775 50  0001 C CNN
+F 3 "" H 1300 3775 50  0001 C CNN
+	1    1300 3775
+	1    0    0    -1
+$EndComp
+Wire Wire Line
+	1150 3575 1300 3575
+Text Label 1150 3575 0    60   ~ 0
+Vin
 $EndSCHEMATC

Commit message: power connector
Parts:
- C17: footprint Capacitors_SMD:C_0402 -> Capacitor_SMD:C_0402_1005Metric
- D6: footprint ptc:DO-214AA -> SMD:DO-214AA
Connections:
- net Q3S: now reaches C17.1, F1.2, Q3.3 (D), Q4.1
Changed lines of the file:
@@
 F 0 "C17" H 2485 5095 35  0000 L CNN
 F 1 "1uF" H 2485 4945 35  0000 L CNN
-F 2 "Capacitors_SMD:C_0402" H 2475 5025 35  0001 C CNN
+F 2 "Capacitor_SMD:C_0402_1005Metric" H 2475 5025 35  0001 C CNN
 F 3 "" H 2475 5025 35  0000 C CNN
 	1    2475 5025
@@
 F 0 "D6" V 3415 5120 35  0000 L CNN
 F 1 "SMBJ5.0A-TR" V 3540 5120 35  0000 L CNN
-F 2 "ptc:DO-214AA" V 3475 5100 35  0001 C CNN
+F 2 "SMD:DO-214AA" V 3475 5100 35  0001 C CNN
 F 3 "" V 3475 5100 35  0001 C CNN
 	1    3475 5100
@@
 Wire Wire Line
 	3475 5200 3475 5275
-Text Label 1910 4875 0    60   ~ 0
+Text Label 1900 4875 0    60   ~ 0
 Vin
 $Comp
@@
 AR Path="/5E98CC69/5EA1B44B/5EA95F9E" Ref="#PWR?"  Part="1"
 AR Path="/5E9C016D/5EA95F9E" Ref="#PWR?"  Part="1"
-AR Path="/5EA61A2E/5EA95F9E" Ref="#PWR?"  Part="1"
-F 0 "#PWR?" H 1300 3525 50  0001 C CNN
+AR Path="/5EA61A2E/5EA95F9E" Ref="#PWR0227"  Part="1"
+F 0 "#PWR0227" H 1300 3525 50  0001 C CNN
 F 1 "GND" H 1305 3602 50  0000 C CNN
 F 2 "" H 1300 3775 50  0001 C CNN
@@
 Text Label 1150 3575 0    60   ~ 0
 Vin
+Text Label 2675 4875 0    50   ~ 0
+Q3S
+Text Label 3200 4875 0    50   ~ 0
+Q3D
 $EndSCHEMATC

Commit message: relayout
Connections:
- net GND: now also PWR1.1 (Pin_1), PWR1.2 (Pin_2); no longer PWR1.5 (Pin_5), PWR1.6 (Pin_6)
- net Vin: now also PWR1.5 (Pin_5), PWR1.6 (Pin_6); no longer PWR1.1 (Pin_1), PWR1.2 (Pin_2)
Changed lines of the file:
@@
 L Connector_Generic:Conn_02x03_Odd_Even G?
 U 1 1 5EAC048F
-P 1500 3675
+P 1600 3675
 AR Path="/5E9C016D/5EAC048F" Ref="G?"  Part="1"
 AR Path="/5EA61A2E/5EAC048F" Ref="PWR1"  Part="1"
-F 0 "PWR1" H 1450 3975 50  0000 L CNN
-F 1 "Conn_01x03" H 1580 3626 50  0001 L CNN
-F 2 "TH:10142708-06200LF" H 1500 3675 50  0001 C CNN
-F 3 "~" H 1500 3675 50  0001 C CNN
-	1    1500 3675
-	1    0    0    -1
+F 0 "PWR1" H 1550 3975 50  0000 L CNN
+F 1 "Conn_01x03" H 1680 3626 50  0001 L CNN
+F 2 "TH:10142708-06200LF" H 1600 3675 50  0001 C CNN
+F 3 "~" H 1600 3675 50  0001 C CNN
+	1    1600 3675
+	-1   0    0    1
 $EndComp
 $Comp
@@
 	1    0    0    -1
 $EndComp
-Wire Wire Line
-	1150 3575 1300 3575
 Text Label 1150 3575 0    60   ~ 0
 Vin
@@
 Text Label 3200 4875 0    50   ~ 0
 Q3D
+Wire Wire Line
+	1150 3575 1300 3575
 $EndSCHEMATC
