File: pcb/Sensors.sch (KiCad schematic (older format))
At the start: 9 parts, among them U1 MPL3115A2, U13 HTS221

Commit message: Added digiKey part number for some components
Parts:
- C15, C31, C32: DigiKey (none) -> 1276-1442-1-ND
- C41, C78: DigiKey (none) -> 1276-1038-1-ND
- R44, R45: DigiKey (none) -> 311-10KJRCT-ND
- U1: DigiKey (none) -> MPL115A2-ND
Changed lines of the file:
@@
 F 2 "Capacitor_SMD:C_0402_1005Metric" H 3250 2425 60  0001 C CNN
 F 3 "" H 3250 2425 60  0000 C CNN
+F 4 "1276-1442-1-ND" H 3250 2425 50  0001 C CNN "DigiKey"
 	1    3250 2425
 	1    0    0    -1
@@
 F 2 "Capacitor_SMD:C_0402_1005Metric" H 3200 4425 60  0001 C CNN
 F 3 "" H 3200 4425 60  0000 C CNN
+F 4 "1276-1442-1-ND" H 3200 4425 50  0001 C CNN "DigiKey"
 	1    3200 4425
 	1    0    0    -1
@@
 F 2 "SMD:8LGA" H 2600 2225 60  0001 C CNN
 F 3 "" H 2600 2225 60  0000 C CNN
+F 4 "MPL115A2-ND" H 2600 2225 50  0001 C CNN "DigiKey"
 	1    2600 2225
 	-1   0    0    -1
@@
 F 2 "Capacitor_SMD:C_0603_1608Metric" H 4225 2300 60  0001 C CNN
 F 3 "" H 4225 2300 60  0000 C CNN
+F 4 "1276-1038-1-ND" H 4225 2300 50  0001 C CNN "DigiKey"
 	1    4225 2300
 	1    0    0    -1
@@
 F 2 "Capacitor_SMD:C_0603_1608Metric" H 3625 4425 60  0001 C CNN
 F 3 "" H 3625 4425 60  0000 C CNN
+F 4 "1276-1038-1-ND" H 3625 4425 50  0001 C CNN "DigiKey"
 	1    3625 4425
 	1    0    0    -1
@@
 F 2 "Capacitor_SMD:C_0402_1005Metric" H 3900 2300 60  0001 C CNN
 F 3 "" H 3900 2300 60  0000 C CNN
+F 4 "1276-1442-1-ND" H 3900 2300 50  0001 C CNN "DigiKey"
 	1    3900 2300
 	1    0    0    -1
@@
 F 2 "Resistor_SMD:R_0402_1005Metric" H 5475 2050 50  0001 C CNN
 F 3 "~" H 5475 2050 50  0001 C CNN
+F 4 "311-10KJRCT-ND" H 5475 2050 50  0001 C CNN "DigiKey"
 	1    5475 2050
 	1    0    0    -1
@@
 F 2 "Resistor_SMD:R_0402_1005Metric" H 5475 2550 50  0001 C CNN
 F 3 "~" H 5475 2550 50  0001 C CNN
+F 4 "311-10KJRCT-ND" H 5475 2550 50  0001 C CNN "DigiKey"
 	1    5475 2550
 	1    0    0    -1
