File: pcb/ElectroValves.sch (KiCad schematic (older format))
At the start: 53 parts, among them P2 Conn_01x04_Female, Q1 PN2222, Q2 PN2222, Q6 PN2222, Q7 PN2222, U11 AQH3223AX, U12 AQH3223AX, U19 AQH3223AX, U20 AQH3223AX, U3 TLP240D, U4 TLP240D, U5 TLP240D, U6 TLP240D, U7 TLP240D, U8 TLP240D

Commit message: Added digiKey part number for some components
Parts:
- P2: DigiKey (none) -> 277-6269-ND; DigiKey2 (none) -> 277-5896-ND
- Q1, Q2, Q6, Q7: DigiKey (none) -> 1727-2956-1-ND
- R16, R17, R18, R19, R20, R21: DigiKey (none) -> P200LCT-ND
- R22, R23, R58, R61: DigiKey (none) -> P330LCT-ND
- R35, R36, R57, R60: DigiKey (none) -> P22JCT-ND
- RJ1: DigiKey (none) -> S2012EC-04-ND; DigiKey2 (none) -> S9337-ND
- RJ2, RJ3, RJ4, RJ5, RJ6: DigiKey (none) -> S2012EC-04-ND
- RL1, RL2, RL3, RL4, RL5, RL6: DigiKey (none) -> 277-1206-ND; DigiKey2 (none) -> 277-1161-ND
- RL10, RL7, RL8, RL9: DigiKey (none) -> 277-1106-ND; DigiKey2 (none) -> 277-1011-ND
Changed lines of the file:
@@
 F 2 "Resistor_SMD:R_0402_1005Metric" V 2330 1600 50  0001 C CNN
 F 3 "~" H 2400 1600 50  0001 C CNN
+F 4 "P200LCT-ND" V 2400 1600 50  0001 C CNN "DigiKey"
 	1    2400 1600
 	0    1    1    0
@@
 F 2 "Resistor_SMD:R_0402_1005Metric" V 4505 1600 50  0001 C CNN
 F 3 "~" H 4575 1600 50  0001 C CNN
+F 4 "P200LCT-ND" V 4575 1600 50  0001 C CNN "DigiKey"
 	1    4575 1600
 	0    1    1    0
@@
 F 2 "Resistor_SMD:R_0402_1005Metric" V 2330 3375 50  0001 C CNN
 F 3 "~" H 2400 3375 50  0001 C CNN
+F 4 "P200LCT-ND" V 2400 3375 50  0001 C CNN "DigiKey"
 	1    2400 3375
 	0    1    1    0
@@
 F 2 "Resistor_SMD:R_0402_1005Metric" V 4505 3425 50  0001 C CNN
 F 3 "~" H 4575 3425 50  0001 C CNN
+F 4 "P200LCT-ND" V 4575 3425 50  0001 C CNN "DigiKey"
 	1    4575 3425
 	0    1    1    0
@@
 F 2 "Resistor_SMD:R_0402_1005Metric" V 2330 5100 50  0001 C CNN
 F 3 "~" H 2400 5100 50  0001 C CNN
+F 4 "P200LCT-ND" V 2400 5100 50  0001 C CNN "DigiKey"
 	1    2400 5100
 	0    1    1    0
@@
 F 2 "Resistor_SMD:R_0402_1005Metric" V 4505 5200 50  0001 C CNN
 F 3 "~" H 4575 5200 50  0001 C CNN
+F 4 "P200LCT-ND" V 4575 5200 50  0001 C CNN "DigiKey"
 	1    4575 5200
 	0    1    1    0
@@
 F 2 "Connector_Phoenix_MC:PhoenixContact_MC_1,5_2-G-3.81_1x02_P3.81mm_Horizontal" H 4025 1500 50  0001 C CNN
 F 3 "~" H 4025 1500 50  0001 C CNN
+F 4 "277-1206-ND" H 4025 1500 50  0001 C CNN "DigiKey"
+F 5 "277-1161-ND" H 4025 1500 50  0001 C CNN "DigiKey2"
 	1    4025 1500
 	1    0    0    -1
@@
 F 2 "SMD:SOT23_Transistor" H 7750 1575 50  0001 L CIN
 F 3 "http://www.fairchildsemi.com/ds/PN/PN2222A.pdf" H 7550 1650 50  0001 L CNN
+F 4 "1727-2956-1-ND" H 7550 1650 50  0001 C CNN "DigiKey"
 	1    7550 1650
 	1    0    0    -1
@@
 F 2 "Resistor_SMD:R_0402_1005Metric" V 7130 1650 50  0001 C CNN
 F 3 "~" H 7200 1650 50  0001 C CNN
+F 4 "P330LCT-ND" V 7200 1650 50  0001 C CNN "DigiKey"
 	1    7200 1650
 	0    1    1    0
@@
 F 2 "Resistor_SMD:R_0402_1005Metric" V 7730 2800 50  0001 C CNN
 F 3 "~" H 7800 2800 50  0001 C CNN
+F 4 "P22JCT-ND" V 7800 2800 50  0001 C CNN "DigiKey"
 	1    7800 2800
 	0    1    1    0
@@
 F 2 "Resistor_SMD:R_0402_1005Metric" V 7130 3000 50  0001 C CNN
 F 3 "~" H 7200 3000 50  0001 C CNN
+F 4 "P330LCT-ND" V 7200 3000 50  0001 C CNN "DigiKey"
 	1    7200 3000
 	0    1    1    0
@@
 F 2 "SMD:SOT23_Transistor" H 7750 2925 50  0001 L CIN
 F 3 "http://www.fairchildsemi.com/ds/PN/PN2222A.pdf" H 7550 3000 50  0001 L CNN
+F 4 "1727-2956-1-ND" H 7550 3000 50  0001 C CNN "DigiKey"
 	1    7550 3000
 	1    0    0    -1
@@
 F 2 "Connector_Phoenix_MC:PhoenixContact_MC_1,5_2-G-3.81_1x02_P3.81mm_Horizontal" H 6200 1500 50  0001 C CNN
 F 3 "~" H 6200 1500 50  0001 C CNN
+F 4 "277-1206-ND" H 6200 1500 50  0001 C CNN "DigiKey"
+F 5 "277-1161-ND" H 6200 1500 50  0001 C CNN "DigiKey2"
 	1    6200 1500
 	1    0    0    -1
@@
 F 2 "Connector_Phoenix_MC:PhoenixContact_MC_1,5_2-G-3.81_1x02_P3.81mm_Horizontal" H 6200 3325 50  0001 C CNN
 F 3 "~" H 6200 3325 50  0001 C CNN
+F 4 "277-1206-ND" H 6200 3325 50  0001 C CNN "DigiKey"
+F 5 "277-1161-ND" H 6200 3325 50  0001 C CNN "DigiKey2"
 	1    6200 3325
 	1    0    0    -1
@@
 F 2 "Connector_Phoenix_MC:PhoenixContact_MC_1,5_2-G-3.81_1x02_P3.81mm_Horizontal" H 4025 5000 50  0001 C CNN
 F 3 "~" H 4025 5000 50  0001 C CNN
+F 4 "277-1206-ND" H 4025 5000 50  0001 C CNN "DigiKey"
+F 5 "277-1161-ND" H 4025 5000 50  0001 C CNN "DigiKey2"
 	1    4025 5000
 	1    0    0    -1
@@
 F 2 "Connector_Phoenix_MC:PhoenixContact_MC_1,5_2-G-3.81_1x02_P3.81mm_Horizontal" H 6200 5100 50  0001 C CNN
 F 3 "~" H 6200 5100 50  0001 C CNN
+F 4 "277-1206-ND" H 6200 5100 50  0001 C CNN "DigiKey"
+F 5 "277-1161-ND" H 6200 5100 50  0001 C CNN "DigiKey2"
 	1    6200 5100
 	1    0    0    -1
@@
 F 2 "Connector_Phoenix_MSTB:PhoenixContact_MSTBA_2,5_2-G-5,08_1x02_P5.08mm_Horizontal" H 10975 2850 50  0001 C CNN
 F 3 "~" H 10975 2850 50  0001 C CNN
+F 4 "277-1106-ND" H 10975 2850 50  0001 C CNN "DigiKey"
+F 5 "277-1011-ND" H 10975 2850 50  0001 C CNN "DigiKey2"
 	1    10975 2850
 	1    0    0    1
@@
 F 2 "Connector_Phoenix_MSTB:PhoenixContact_MSTBA_2,5_2-G-5,08_1x02_P5.08mm_Horizontal" H 10975 1500 50  0001 C CNN
 F 3 "~" H 10975 1500 50  0001 C CNN
+F 4 "277-1106-ND" H 10975 1500 50  0001 C CNN "DigiKey"
+F 5 "277-1011-ND" H 10975 1500 50  0001 C CNN "DigiKey2"
 	1    10975 1500
 	1    0    0    1
@@
 F 2 "Connector_Phoenix_MC:PhoenixContact_MC_1,5_2-G-3.81_1x02_P3.81mm_Horizontal" H 4025 3275 50  0001 C CNN
 F 3 "~" H 4025 3275 50  0001 C CNN
+F 4 "277-1206-ND" H 4025 3275 50  0001 C CNN "DigiKey"
+F 5 "277-1161-ND" H 4025 3275 50  0001 C CNN "DigiKey2"
 	1    4025 3275
 	1    0    0    -1
@@
 F 2 "Resistor_SMD:R_0402_1005Metric" V 7730 1450 50  0001 C CNN
 F 3 "~" H 7800 1450 50  0001 C CNN
+F 4 "P22JCT-ND" V 7800 1450 50  0001 C CNN "DigiKey"
 	1    7800 1450
 	0    1    1    0
@@
 F 2 "Connector_Phoenix_MSTB:PhoenixContact_MSTB_2,5_2-GF_1x02_P5.00mm_Horizontal_ThreadedFlange_MountHole" H 9200 6250 50  0001 C CNN
 F 3 "~" H 9200 6250 50  0001 C CNN
+F 4 "277-6269-ND" H 9200 6250 50  0001 C CNN "DigiKey"
+F 5 "277-5896-ND" H 9200 6250 50  0001 C CNN "DigiKey2"
 	1    9200 6250
 	1    0    0    1
@@
 F 2 "Connector_PinHeader_2.54mm:PinHeader_2x04_P2.54mm_Vertical" H 3550 1300 50  0001 C CNN
 F 3 "~" H 3550 1300 50  0001 C CNN
+F 4 "S2012EC-04-ND" V 3550 1300 50  0001 C CNN "DigiKey"
+F 5 "S9337-ND" V 3550 1300 50  0001 C CNN "DigiKey2"
 	1    3550 1300
 	0    1    -1   0
@@
 F 2 "Connector_PinHeader_2.54mm:PinHeader_2x04_P2.54mm_Vertical" H 5725 1300 50  0001 C CNN
 F 3 "~" H 5725 1300 50  0001 C CNN
+F 4 "S2012EC-04-ND" V 5725 1300 50  0001 C CNN "DigiKey"
 	1    5725 1300
 	0    1    -1   0
@@
 F 2 "Connector_PinHeader_2.54mm:PinHeader_2x04_P2.54mm_Vertical" H 3550 3075 50  0001 C CNN
 F 3 "~" H 3550 3075 50  0001 C CNN
+F 4 "S2012EC-04-ND" V 3550 3075 50  0001 C CNN "DigiKey"
 	1    3550 3075
 	0    1    -1   0
@@
 F 2 "Connector_PinHeader_2.54mm:PinHeader_2x04_P2.54mm_Vertical" H 5725 3125 50  0001 C CNN
 F 3 "~" H 5725 3125 50  0001 C CNN
+F 4 "S2012EC-04-ND" V 5725 3125 50  0001 C CNN "DigiKey"
 	1    5725 3125
 	0    1    -1   0
@@
 F 2 "Connector_PinHeader_2.54mm:PinHeader_2x04_P2.54mm_Vertical" H 3550 4800 50  0001 C CNN
 F 3 "~" H 3550 4800 50  0001 C CNN
+F 4 "S2012EC-04-ND" V 3550 4800 50  0001 C CNN "DigiKey"
 	1    3550 4800
 	0    1    -1   0
@@
 F 2 "Connector_PinHeader_2.54mm:PinHeader_2x04_P2.54mm_Vertical" H 5725 4900 50  0001 C CNN
 F 3 "~" H 5725 4900 50  0001 C CNN
+F 4 "S2012EC-04-ND" V 5725 4900 50  0001 C CNN "DigiKey"
 	1    5725 4900
 	0    1    -1   0
@@
 F 2 "SMD:SOT23_Transistor" H 7775 4225 50  0001 L CIN
 F 3 "http://www.fairchildsemi.com/ds/PN/PN2222A.pdf" H 7575 4300 50  0001 L CNN
+F 4 "1727-2956-1-ND" H 7575 4300 50  0001 C CNN "DigiKey"
 	1    7575 4300
 	1    0    0    -1
@@
 F 2 "Resistor_SMD:R_0402_1005Metric" V 7155 4300 50  0001 C CNN
 F 3 "~" H 7225 4300 50  0001 C CNN
+F 4 "P330LCT-ND" V 7225 4300 50  0001 C CNN "DigiKey"
 	1    7225 4300
 	0    1    1    0
@@
 F 2 "Resistor_SMD:R_0402_1005Metric" V 7755 5450 50  0001 C CNN
 F 3 "~" H 7825 5450 50  0001 C CNN
+F 4 "P22JCT-ND" V 7825 5450 50  0001 C CNN "DigiKey"
 	1    7825 5450
 	0    1    1    0
@@
 F 2 "Resistor_SMD:R_0402_1005Metric" V 7155 5650 50  0001 C CNN
 F 3 "~" H 7225 5650 50  0001 C CNN
+F 4 "P330LCT-ND" V 7225 5650 50  0001 C CNN "DigiKey"
 	1    7225 5650
 	0    1    1    0
@@
 F 2 "SMD:SOT23_Transistor" H 7775 5575 50  0001 L CIN
 F 3 "http://www.fairchildsemi.com/ds/PN/PN2222A.pdf" H 7575 5650 50  0001 L CNN
+F 4 "1727-2956-1-ND" H 7575 5650 50  0001 C CNN "DigiKey"
 	1    7575 5650
 	1    0    0    -1
@@
 F 2 "Connector_Phoenix_MSTB:PhoenixContact_MSTBA_2,5_2-G-5,08_1x02_P5.08mm_Horizontal" H 11000 5500 50  0001 C CNN
 F 3 "~" H 11000 5500 50  0001 C CNN
+F 4 "277-1106-ND" H 11000 5500 50  0001 C CNN "DigiKey"
+F 5 "277-1011-ND" H 11000 5500 50  0001 C CNN "DigiKey2"
 	1    11000 5500
 	1    0    0    1
@@
 F 2 "Connector_Phoenix_MSTB:PhoenixContact_MSTBA_2,5_2-G-5,08_1x02_P5.08mm_Horizontal" H 11000 4150 50  0001 C CNN
 F 3 "~" H 11000 4150 50  0001 C CNN
+F 4 "277-1106-ND" H 11000 4150 50  0001 C CNN "DigiKey"
+F 5 "277-1011-ND" H 11000 4150 50  0001 C CNN "DigiKey2"
 	1    11000 4150
 	1    0    0    1
@@
 F 2 "Resistor_SMD:R_0402_1005Metric" V 7755 4100 50  0001 C CNN
 F 3 "~" H 7825 4100 50  0001 C CNN
+F 4 "P22JCT-ND" V 7825 4100 50  0001 C CNN "DigiKey"
 	1    7825 4100
 	0    1    1    0

Commit message: Added all references on silkscreen added BOM for sensor modules
Parts:
- U11, U19, U20: DigiKey (none) -> 255-6003-1-ND; Digikey 255-6003-1-ND -> (none)
Changed lines of the file:
@@
 F 2 "SMD:AQH3223A" H 8850 990 60  0001 C CNN
 F 3 "https://b2b-api.panasonic.eu/file_stream/pids/fileversion/2787" H 7950 750 60  0001 C CNN
-F 4 "255-6003-1-ND" H 7950 750 50  0001 C CNN "Digikey"
+F 4 "255-6003-1-ND" H 7950 750 50  0001 C CNN "DigiKey"
 	1    7950 750
 	1    0    0    -1
@@
 F 2 "SMD:AQH3223A" H 8875 3640 60  0001 C CNN
 F 3 "https://b2b-api.panasonic.eu/file_stream/pids/fileversion/2787" H 7975 3400 60  0001 C CNN
-F 4 "255-6003-1-ND" H 7975 3400 50  0001 C CNN "Digikey"
+F 4 "255-6003-1-ND" H 7975 3400 50  0001 C CNN "DigiKey"
 	1    7975 3400
 	1    0    0    -1
@@
 F 2 "SMD:AQH3223A" H 8875 4990 60  0001 C CNN
 F 3 "https://b2b-api.panasonic.eu/file_stream/pids/fileversion/2787" H 7975 4750 60  0001 C CNN
-F 4 "255-6003-1-ND" H 7975 4750 50  0001 C CNN "Digikey"
+F 4 "255-6003-1-ND" H 7975 4750 50  0001 C CNN "DigiKey"
 	1    7975 4750
 	1    0    0    -1
