File: ABPDANT060MGAA5_sensor/ABPDANT060MGAA5_sensor_module.sch (KiCad schematic (older format))
At the start: 9 parts, among them J1 Conn_02x04_Odd_Even, J2 Conn_02x07_Odd_Even, U1 ABPDANT060MGAA5, U2 LM358

Commit message: Added DigiKey part number to J2 connector WM17456-ND
Parts:
- J1, J2: DigiKey (none) -> WM17456-ND
Changed lines of the file:
@@
 F 2 "Connector_PinHeader_2.54mm:PinHeader_2x04_P2.54mm_Vertical_SMD" H 4950 1825 50  0001 C CNN
 F 3 "~" H 4950 1825 50  0001 C CNN
+F 4 "WM17456-ND" H 4950 1825 50  0001 C CNN "DigiKey"
 	1    4950 1825
 	1    0    0    -1
@@
 F 2 "Connector_PinHeader_2.54mm:PinHeader_2x07_P2.54mm_Vertical_SMD" H 2350 1875 50  0001 C CNN
 F 3 "~" H 2350 1875 50  0001 C CNN
+F 4 "WM17456-ND" H 2350 1875 50  0001 C CNN "DigiKey"
 	1    2350 1875
 	1    0    0    -1

Commit message: Added capacitors DigiKey part number
Parts:
- C1, C3: DigiKey (none) -> 732-7939-1-ND
- C2: DigiKey (none) -> 311-4053-1-ND
Changed lines of the file:
@@
 F 2 "Capacitor_SMD:C_0603_1608Metric" H 1763 3725 50  0001 C CNN
 F 3 "~" H 1725 3875 50  0001 C CNN
+F 4 "732-7939-1-ND" H 1725 3875 50  0001 C CNN "DigiKey"
 	1    1725 3875
 	1    0    0    -1
@@
 F 2 "Capacitor_SMD:C_0603_1608Metric" H 3113 3325 50  0001 C CNN
 F 3 "~" H 3075 3475 50  0001 C CNN
+F 4 "311-4053-1-ND" H 3075 3475 50  0001 C CNN "DigiKey"
 	1    3075 3475
 	1    0    0    -1
@@
 F 2 "Capacitor_SMD:C_0603_1608Metric" H 4913 2975 50  0001 C CNN
 F 3 "~" H 4875 3125 50  0001 C CNN
+F 4 "732-7939-1-ND" H 4875 3125 50  0001 C CNN "DigiKey"
 	1    4875 3125
 	1    0    0    -1

Commit message: Added all references on silkscreen added BOM for sensor modules
Parts:
- J1: DigiKey WM17456-ND -> 609-6367-ND
- J2: DigiKey WM17456-ND -> 609-6365-ND
Changed lines of the file:
@@
 F 2 "Connector_PinHeader_2.54mm:PinHeader_2x04_P2.54mm_Vertical_SMD" H 4950 1825 50  0001 C CNN
 F 3 "~" H 4950 1825 50  0001 C CNN
-F 4 "WM17456-ND" H 4950 1825 50  0001 C CNN "DigiKey"
+F 4 "609-6367-ND" H 4950 1825 50  0001 C CNN "DigiKey"
 	1    4950 1825
 	1    0    0    -1
@@
 F 2 "Connector_PinHeader_2.54mm:PinHeader_2x07_P2.54mm_Vertical_SMD" H 2350 1875 50  0001 C CNN
 F 3 "~" H 2350 1875 50  0001 C CNN
-F 4 "WM17456-ND" H 2350 1875 50  0001 C CNN "DigiKey"
+F 4 "609-6365-ND" H 2350 1875 50  0001 C CNN "DigiKey"
 	1    2350 1875
 	1    0    0    -1
