File: ABPDJJT001PDSA3_sensor/ABPDJJT001PDSA3_sensor_module.sch (KiCad schematic (older format))
At the start: 4 parts, among them J1 Conn_02x04_Odd_Even, J2 Conn_02x07_Odd_Even, U1 ABPDJJ001PDSA3

Commit message: Added all references on silkscreen added BOM for sensor modules
Parts:
- C1: DigiKey (none) -> 1276-1258-1-ND
- J1: DigiKey (none) -> 609-6367-ND
- J2: DigiKey (none) -> 609-6365-ND
Changed lines of the file:
@@
 F 2 "Connector_PinHeader_2.54mm:PinHeader_2x04_P2.54mm_Vertical_SMD" H 4950 1825 50  0001 C CNN
 F 3 "~" H 4950 1825 50  0001 C CNN
+F 4 "609-6367-ND" H 4950 1825 50  0001 C CNN "DigiKey"
 	1    4950 1825
 	1    0    0    -1
@@
 F 2 "Connector_PinHeader_2.54mm:PinHeader_2x07_P2.54mm_Vertical_SMD" H 2350 1875 50  0001 C CNN
 F 3 "~" H 2350 1875 50  0001 C CNN
+F 4 "609-6365-ND" H 2350 1875 50  0001 C CNN "DigiKey"
 	1    2350 1875
 	1    0    0    -1
@@
 F 2 "Capacitor_SMD:C_0603_1608Metric" H 1663 3100 50  0001 C CNN
 F 3 "~" H 1625 3250 50  0001 C CNN
+F 4 "1276-1258-1-ND" H 1625 3250 50  0001 C CNN "DigiKey"
 	1    1625 3250
 	1    0    0    -1
