File: pcb_2.0/power_stepper.sch (KiCad schematic (older format))
At the start: 51 parts, among them J2 1757284, SW1 SW_DIP_x01, U16 UCC12040, U17 ISO7762, U2 powerSTEP01

Commit message: driver for motor eliminated
Parts:
- removed C1: 22uF, Capacitor_SMD:C_0805_2012Metric, symbol Device:CP
- removed C10, C11: 100uF 100V (Low ESR), Capacitor_THT:CP_Radial_D12.5mm_P5.00mm, symbol Device:CP
- removed C12, C22: 0.1uF, Capacitor_SMD:C_0402_1005Metric, symbol Device:C
- removed C13: 47nF 100V, Capacitor_SMD:C_0805_2012Metric, symbol Device:C
- removed C14, C34, C35, C37, C74: 0.1uF, Capacitor_SMD:C_0402_1005Metric, symbol Device:C_Small
- removed C2, C3: 470nF 100V, Capacitor_SMD:C_0805_2012Metric, symbol Device:C
- removed C33, C36: 10uF, Capacitor_SMD:C_0603_1608Metric, symbol Device:C_Small
- removed C4: 220nF, Capacitor_SMD:C_0402_1005Metric, symbol Device:C
- removed C5: 0.1uF, Capacitor_SMD:C_0603_1608Metric, symbol Device:C
- removed C6, C7, C8, C9: 220nF 100V, Capacitor_SMD:C_0805_2012Metric, symbol Device:C
- removed D0: 80V (Back EMF Clamp), Diode_SMD:D_SMB, symbol Device:D_Schottky
- removed D1: D_Schottky_x2_Serial_AKC, Package_TO_SOT_SMD:SOT-23, symbol Device:D_Schottky_x2_Serial_AKC
- removed D2: D_Schottky, Diode_SMD:D_SOD-123, symbol Device:D_Schottky
- removed D3: LED GRN, Diode_SMD:D_0603_1608Metric, symbol Device:LED
- removed D5: LED RED, Diode_SMD:D_0603_1608Metric, symbol Device:LED
- removed J2: 1757284, Connector_Phoenix_MSTB:PhoenixContact_MSTBA_2,5_6-G-5,08_1x06_P5.08mm_Horizontal, symbol Connector:Screw_Terminal_01x06
- removed JP1, JP2: Jumper_2_Open, Klofas-Connectors:STpowerSTEP01_JMP, symbol Jumper:Jumper_2_Open
- removed JP4: SolderJumper_3_Bridged12, Jumper:SolderJumper-3_P1.3mm_Bridged12_RoundedPad1.0x1.5mm, symbol Jumper:SolderJumper_3_Bridged12
- removed R1: -, Klofas-Passives:Resistor_NP_0805, symbol Device:R
- removed R11: 1k, Resistor_SMD:R_0402_1005Metric, symbol Device:R
- removed R3: 47K, Resistor_SMD:R_0603_1608Metric, symbol Device:R
- removed R39: 100k, Resistor_SMD:R_0402_1005Metric, symbol Device:R_Small
- removed R4: 1.8K, Resistor_SMD:R_0603_1608Metric, symbol Device:R
- removed R63: 10k, Resistor_SMD:R_0402_1005Metric, symbol Device:R
- removed R7, R8: 39K, Resistor_SMD:R_0402_1005Metric, symbol Device:R
- removed R9: 330, Resistor_SMD:R_0402_1005Metric, symbol Device:R
- removed RS1, RS2, RS3, RS4, RS5, RS6, RS7, RS8: 0.27, Resistor_SMD:R_2512_6332Metric, symbol Device:R
- removed SW1: SW_DIP_x01, Connector_Molex:Molex_CLIK-Mate_502443-0270_1x02-1MP_P2.00mm_Vertical, symbol Switch:SW_DIP_x01
- removed U16: UCC12040, Package_SO:SOIC-16W_7.5x10.3mm_P1.27mm, symbol UCC12040:UCC12040
- removed U17: ISO7762, Package_SO:SSOP-16_3.9x4.9mm_P0.635mm, symbol ISO7762:ISO7762
- removed U2: powerSTEP01, SMD:powerSTEP01, symbol powerstep01:powerSTEP01-Klofas
Connections:
- no-connect marks 3 -> 0
Other:
- note removed: "SW N.C."
