File: ABPDANT015PGAA5_sensor/ABPDANT015PGAA5_sensor_module.sch (KiCad schematic (older format))
At the start: 9 parts, among them J1 Conn_02x04_Odd_Even, J2 Conn_02x07_Odd_Even, U1 ABPDANT060MGAA5, U2 LM358

Commit message: Added DigiKey part number
Parts:
- C1, C3: DigiKey (none) -> 732-7939-1-ND
- C2: DigiKey (none) -> 311-4053-1-ND
Changed lines of the file:
@@
 F 2 "Capacitor_SMD:C_0603_1608Metric" H 1763 3725 50  0001 C CNN
 F 3 "~" H 1725 3875 50  0001 C CNN
+F 4 "732-7939-1-ND" H 1725 3875 50  0001 C CNN "DigiKey"
 	1    1725 3875
 	1    0    0    -1
@@
 F 2 "Capacitor_SMD:C_0603_1608Metric" H 3113 3325 50  0001 C CNN
 F 3 "~" H 3075 3475 50  0001 C CNN
+F 4 "311-4053-1-ND" H 3075 3475 50  0001 C CNN "DigiKey"
 	1    3075 3475
 	1    0    0    -1
@@
 F 2 "Capacitor_SMD:C_0603_1608Metric" H 4913 2975 50  0001 C CNN
 F 3 "~" H 4875 3125 50  0001 C CNN
+F 4 "732-7939-1-ND" H 4875 3125 50  0001 C CNN "DigiKey"
 	1    4875 3125
 	1    0    0    -1

Commit message: Added BOM for PCB ABPDANT015PGAA5 sensor
Parts:
- J1: DigiKey (none) -> 609-6367-ND
- J2: DigiKey (none) -> 609-6365-ND
Changed lines of the file:
@@
 F 2 "Connector_PinHeader_2.54mm:PinHeader_2x04_P2.54mm_Vertical_SMD" H 4950 1825 50  0001 C CNN
 F 3 "~" H 4950 1825 50  0001 C CNN
+F 4 "609-6367-ND" H 4950 1825 50  0001 C CNN "DigiKey"
 	1    4950 1825
 	1    0    0    -1
@@
 F 2 "Connector_PinHeader_2.54mm:PinHeader_2x07_P2.54mm_Vertical_SMD" H 2350 1875 50  0001 C CNN
 F 3 "~" H 2350 1875 50  0001 C CNN
+F 4 "609-6365-ND" H 2350 1875 50  0001 C CNN "DigiKey"
 	1    2350 1875
 	1    0    0    -1

Commit message: Position for J2 U1 and U2 modified
Parts:
- U2: footprint (none) -> Package_SO:TSSOP-8_4.4x3mm_P0.65mm
Changed lines of the file:
@@
 F 0 "U2" H 3833 3421 50  0000 L CNN
 F 1 "LM358" H 3833 3330 50  0000 L CNN
-F 2 "" H 3875 3375 50  0001 C CNN
+F 2 "Package_SO:TSSOP-8_4.4x3mm_P0.65mm" H 3875 3375 50  0001 C CNN
 F 3 "http://www.ti.com/lit/ds/symlink/lm2904-n.pdf" H 3875 3375 50  0001 C CNN
 	3    3875 3375
