File: sensor_oxigeno/sensor_oxigeno.kicad_pcb (KiCad board)
At the start: 4 copper layers, 29 x 35 mm, 12 parts, among them J1 Conn_01x02_Female, J2 Conn_02x07_Odd_Even, J3 Conn_02x04_Odd_Even, U1 LM318N, U2 INA128

Commit message: Gerber files created
Routing:
- added copper zone on F.Cu, net GND
